Commit message: modified urdf to match image

File: moveit_tutorial/urdf/robot.urdf (robot description, URDF)
Before this commit: robot custom_robot, 2 links, 2 joints
Links:
- removed link base_link
- removed link link1
- added link my_link1
- added link my_link2
Joints:
- removed joint base_joint
- removed joint joint1
- added joint my_joint1: type continuous, parent my_link1, child my_link2, origin xyz=0 0 0.5 rpy=0 0 0, axis 1 0 0
