Commit message: Added frame to end-effector to match world

File: moveit_tutorial/urdf/ur_demo_description.urdf.xacro (robot description, xacro)
@@ -28,3 +28,9 @@
 		<origin xyz="0.14 -0.76 1.22" rpy="0 ${pi/2 - 20 * pi/180} ${pi/2}"/>
 	</joint>
+   	<link name="ee_link_mod"/>
+	<joint name="ee_joint_mod" type="fixed">
+		<parent link="ee_link"/>
+		<child link="ee_link_mod"/>
+		<origin xyz=" 0 0 0" rpy="0 ${-pi/2} 0"/>
+	</joint>
 </robot>
