Commit message: added end-effector frame to match world

File: moveit_tutorial/urdf/denso_demo_description.urdf.xacro (robot description, xacro)
@@ -24,3 +24,9 @@
 		<origin xyz="0.27 0.9 1.23" rpy="0 ${pi/2 - 15 * pi/180} ${-pi/2}"/>
 	</joint>
+	<link name="ee_link_mod"/>
+	<joint name="ee_joint_mod" type="fixed">
+		<parent link="link_6"/>
+		<child link="ee_link_mod"/>
+		<origin xyz=" 0 0 0" rpy="0 ${pi} 0"/>
+	</joint>
 </robot>

Commit message: Added ar tags support to the simulation

File: moveit_tutorial/urdf/denso_demo_description.urdf.xacro (robot description, xacro)
@@ -4,5 +4,6 @@
   <!--xacro:include filename="$(find ur_description)/urdf/common.gazebo.xacro" /-->
   <xacro:include filename="$(find tutorial_commons)/urdf/table_denso.urdf.xacro" />
-  <!--xacro:include filename="$(find tutorial_commons)/urdf/kinect.xacro"/-->
+  <xacro:include filename="$(find tutorial_commons)/urdf/kinect.xacro"/>
+  <xacro:property name="sim" value="$(arg sim)"/>
 	<link name="world"/>
 	<!-- include platform -->
@@ -14,14 +15,4 @@
  	  <origin xyz="0 0 0" rpy="0 0 0" />
     </xacro:vs087>
-	<!-- include camera -->
-	<!--xacro:sensor_kinect parent="world">
-	  <origin xyz="0.27 0.9 1.22" rpy="0 ${pi/2 - 20 * pi/180} ${-pi/2}"/>
-	</xacro:sensor_kinect-->
-	<link name="camera_link"/>
-	<joint name="camera_joint" type="fixed">
-		<parent link="world"/>
-		<child link="camera_link"/>
-		<origin xyz="0.27 0.9 1.23" rpy="0 ${pi/2 - 15 * pi/180} ${-pi/2}"/>
-	</joint>
 	<link name="ee_link_mod"/>
 	<joint name="ee_joint_mod" type="fixed">
@@ -30,3 +21,17 @@
 		<origin xyz=" 0 0 0" rpy="0 ${pi} 0"/>
 	</joint>
+	<xacro:if value="${sim}">
+	  <xacro:sensor_kinect parent="world">
+	    <origin xyz="0.27 0.9 1.23" rpy="0 ${pi/2 - 15 * pi/180} ${-pi/2}"/>
+	  </xacro:sensor_kinect>
+	</xacro:if>
+	<!-- include camera -->
+	<xacro:unless value="${sim}">
+	  <link name="camera_link"/>
+	  <joint name="camera_joint" type="fixed">
+		<parent link="world"/>
+		<child link="camera_link"/>
+		<origin xyz="0.27 0.9 1.23" rpy="0 ${pi/2 - 15 * pi/180} ${-pi/2}"/>
+	  </joint>
+	</xacro:unless>
 </robot>

File: moveit_tutorial/urdf/ur_demo_description.urdf.xacro (robot description, xacro)
@@ -3,28 +3,19 @@
   <xacro:include filename="$(find ur_description)/urdf/ur5.urdf.xacro" />
   <xacro:include filename="$(find ur_description)/urdf/common.gazebo.xacro" />
- 	<xacro:include filename="$(find tutorial_commons)/urdf/table_ur.urdf.xacro" />
- 	<!--xacro:include filename="$(find tutorial_commons)/urdf/kinect.xacro"/-->
+  <xacro:include filename="$(find tutorial_commons)/urdf/table_ur.urdf.xacro" />
+  <xacro:include filename="$(find tutorial_commons)/urdf/kinect.xacro"/>
+  <xacro:property name="sim" value="$(arg sim)"/>
 	<!-- setup empty world -->
 	<link name="world"/>
 	<!-- include platform -->
 	<xacro:table prefix="" parent="world">
-  	<origin xyz="-0.24 -0.78 -0.75" rpy="0 0 0"/>
+  	  <origin xyz="-0.24 -0.78 -0.75" rpy="0 0 0"/>
 	</xacro:table>
-  <!-- arm -->
+  	<!-- arm -->
 	<xacro:ur5_robot prefix="" joint_limited="true"/>
 	<joint name="world_joint" type="fixed">
-  	<parent link="world" />
-  	<child link = "base_link" />
-  	<origin xyz="0.0 0.0 0.0" rpy="0.0 0.0 ${pi}" />
-	</joint>
-	<!-- include camera -->
-	<!--xacro:sensor_kinect parent="world">
-	<origin xyz="0.5 0 1.089" rpy="${5 * pi/180} ${10 * pi/180} 0"/>
-	</xacro:sensor_kinect-->
-	<link name="camera_link"/>
-	<joint name="camera_joint" type="fixed">
-		<parent link="world"/>
-		<child link="camera_link"/>
-		<origin xyz="0.14 -0.76 1.22" rpy="0 ${pi/2 - 20 * pi/180} ${pi/2}"/>
+  	  <parent link="world" />
+  	  <child link = "base_link" />
+  	  <origin xyz="0.0 0.0 0.0" rpy="0.0 0.0 ${pi}" />
 	</joint>
    	<link name="ee_link_mod"/>
@@ -34,3 +25,17 @@
 		<origin xyz=" 0 0 0" rpy="0 ${-pi/2} 0"/>
 	</joint>
+	<!-- include camera -->
+	<xacro:if value="${sim}">
+	  <xacro:sensor_kinect parent="world">
+		<origin xyz="0.14 -0.76 1.22" rpy="0 ${pi/2 - 20 * pi/180} ${pi/2}"/>
+	  </xacro:sensor_kinect>
+	</xacro:if>
+	<xacro:unless value="${sim}">
+	  <link name="camera_link"/>
+	  <joint name="camera_joint" type="fixed">
+		<parent link="world"/>
+		<child link="camera_link"/>
+		<origin xyz="0.14 -0.76 1.22" rpy="0 ${pi/2 - 20 * pi/180} ${pi/2}"/>
+	  </joint>
+	</xacro:unless>
 </robot>

File: tutorial_commons/urdf/kinect.xacro (robot description, xacro)
@@ -35,7 +35,7 @@
     <origin xyz="0 0 0" rpy="0 0 0"/>
     <parent link="camera_rgb_frame"/>
-    <child link="camera"/>
+    <child link="camera_link"/>
   </joint>
-    <link name="camera">
+    <link name="camera_link">
     <visual>
      <origin xyz="0 0 0" rpy="0 0 ${M_PI/2}"/>
@@ -89,6 +89,6 @@
     </inertial>
 	</link>
-    <gazebo reference="camera">
-      <sensor type="depth" name="camera">
+    <gazebo reference="camera_link">
+      <sensor type="depth" name="camera_link">
         <always_on>true</always_on>
         <update_rate>20.0</update_rate>

Commit message: Stuttgart 19th Feb 2018

File: moveit_tutorial/urdf/denso_demo_description.urdf.xacro (robot description, xacro)
@@ -5,4 +5,5 @@
   <xacro:include filename="$(find tutorial_commons)/urdf/table_denso.urdf.xacro" />
   <xacro:include filename="$(find tutorial_commons)/urdf/kinect.xacro"/>
+	<xacro:arg name="sim" default="true"/>
   <xacro:property name="sim" value="$(arg sim)"/>
 	<link name="world"/>

File: moveit_tutorial/urdf/ur_demo_description.urdf.xacro (robot description, xacro)
@@ -5,4 +5,5 @@
   <xacro:include filename="$(find tutorial_commons)/urdf/table_ur.urdf.xacro" />
   <xacro:include filename="$(find tutorial_commons)/urdf/kinect.xacro"/>
+  <xacro:arg name="sim" default="true"/>
   <xacro:property name="sim" value="$(arg sim)"/>
 	<!-- setup empty world -->
@@ -36,5 +37,5 @@
 		<parent link="world"/>
 		<child link="camera_link"/>
-		<origin xyz="0.14 -0.76 1.22" rpy="0 ${pi/2 - 20 * pi/180} ${pi/2}"/>
+		<origin xyz="0.08 -0.78 1.28" rpy="0 ${pi/2 - 20 * pi/180} ${pi/2}"/>
 	  </joint>
 	</xacro:unless>
